File: Seahorse_v2/seahorse_v2_0_0.kicad_sch (KiCad schematic)
At the start: 82 parts, among them J2 battery_conn_r, J3 track_point_left, J4 niceview_left, J5 niceview_right, J6 track_point_right, SW1 SW_Push, SW10 SW_Push, SW10_r1 SW_Push, SW11 SW_Push, SW11_r1 SW_Push, SW12 SW_Push, SW12_r1 SW_Push, SW13 SW_Push, SW13_r1 SW_Push, SW14 SW_Push, SW14_r1 SW_Push, SW15 SW_Push, SW15_r1 SW_Push, SW16 SW_Push, SW16_r1 SW_Push, SW17 SW_Push, SW17_r1 SW_Push, SW1_r1 SW_Push, SW2 SW_Push, SW2_r1 SW_Push, SW3 SW_Push, SW3_r1 SW_Push, SW4 SW_Push, SW4_r1 SW_Push, SW5 SW_Push, SW5_r1 SW_Push, SW6 SW_Push, SW6_r1 SW_Push, SW7 SW_Push, SW7_r1 SW_Push, SW8 SW_Push, SW8_r1 SW_Push, SW9 SW_Push, SW9_r1 SW_Push, U1 ProMicro-kbd, U2 ProMicro-kbd

Commit message: wip: start on Loce Alda
Parts:
- removed BT1: 1044, 1044:BAT_1044, symbol 1044:1044
- added Bat+1, BatGND1: MountingHole_Pad, kbd:1pin_conn, symbol Mechanical:MountingHole_Pad
- added J1: Battery_conn, Connector_JST:JST_PH_S2B-PH-K_1x02_P2.00mm_Horizontal, symbol Connector:Conn_01x02_Female
- added J7: VIK_Left, Connector_FFC-FPC:Hirose_FH12-12S-0.5SH_1x12-1MP_P0.50mm_Horizontal, symbol Connector:Conn_01x12_Socket
- added J8: VIK_Right, Connector_FFC-FPC:Hirose_FH12-12S-0.5SH_1x12-1MP_P0.50mm_Horizontal, symbol Connector:Conn_01x12_Socket
Connections:
- net BT+: now also Bat+1.1, J1.2 (Pin_2)
- net CS: now also J7.10 (Pin_10)
- net CS_r: now also J8.10 (Pin_10)
- net GPIO1: now also J7.7 (Pin_7)
- net GPIO1_r: now also J8.7 (Pin_7)
- net GPIO2: now also J7.9 (Pin_9)
- net GPIO2_r: now also J8.9 (Pin_9)
- net IPD_CLK: now also J7.4 (Pin_4)
- net IPD_CLK_r: now also J8.4 (Pin_4)
- net IPD_DATA: now also J7.3 (Pin_3)
- net IPD_DATA_r: now also J8.3 (Pin_3)
- net IPD_RST: now also J7.5 (Pin_5)
- net IPD_RST_r: now also J8.5 (Pin_5)
- net MISO: now also J7.11 (Pin_11)
- net MISO_r: now also J8.11 (Pin_11)
- net MOSI: now also J7.8 (Pin_8)
- net MOSI_r: now also J8.8 (Pin_8)
- net SCK: now also J7.12 (Pin_12)
- net SCK_r: now also J8.12 (Pin_12)
- net gnd: now also BatGND1.1, J1.1 (Pin_1), J7.2 (Pin_2)
- net gnd_r: now also J8.2 (Pin_2)
- net vcc: now also J7.1 (Pin_1), J7.6 (Pin_6)
- net vcc_r: now also J8.1 (Pin_1), J8.6 (Pin_6)
