File: loce_alda_v1/loce_alda_v1_0_0.kicad_pcb (KiCad board)
At the start: 2 copper layers, 246.8 x 97.3 mm, 88 parts, among them J1 Battery_conn, J2 battery_conn_r, J3 track_point_left, J4 niceview_left, J5 niceview_right, J6 track_point_right, J7 VIK_Left, J8 VIK_Right, SW1 SW_Push, SW10 SW_Push, SW10_r1 SW_Push, SW11 SW_Push, SW11_r1 SW_Push, SW12 SW_Push, SW12_r1 SW_Push, SW13 SW_Push, SW13_r1 SW_Push, SW14 SW_Push, SW14_r1 SW_Push, SW15 SW_Push, SW15_r1 SW_Push, SW16 SW_Push, SW16_r1 SW_Push, SW17 SW_Push, SW17_r1 SW_Push, SW1_r1 SW_Push, SW2 SW_Push, SW2_r1 SW_Push, SW3 SW_Push, SW3_r1 SW_Push, SW4 SW_Push, SW4_r1 SW_Push, SW5 SW_Push, SW5_r1 SW_Push, SW6 SW_Push, SW6_r1 SW_Push, SW7 SW_Push, SW7_r1 SW_Push, SW8 SW_Push, SW8_r1 SW_Push, SW9 SW_Push, SW9_r1 SW_Push, U1 ProMicro-kbd, U2 ProMicro-kbd

Commit message: wip: start on Loce Alda
Parts:
- removed J2: battery_conn_r, Connector_JST:JST_PH_S2B-PH-K_1x02_P2.00mm_Horizontal
- removed J7: VIK_Left, Connector_FFC-FPC:Hirose_FH12-12S-0.5SH_1x12-1MP_P0.50mm_Horizontal
- removed J8: VIK_Right, Connector_FFC-FPC:Hirose_FH12-12S-0.5SH_1x12-1MP_P0.50mm_Horizontal
- removed U2: ProMicro-kbd, Arduino:Sparkfun_Pro_Micro
- added BT1: 1044, 1044:BAT_1044, F.Cu at (-71.6, 66.2)
- added U3: Seeed Studio XIAO SAMD21, xiao:XIAO-nRF52840-SMD, F.Cu at (9.66, 12.1)
- moved RSW2 36.8 mm to (13.5, 83.5)
- moved J5 25.9 mm to (15.2, 99.5)
Connections:
- J5 pad 5: CS_r -> CS_R
Routing:
- net gnd: track 194.5 -> 0.00 mm, vias 2 -> 0
- net gnd_r: track 183.4 -> 0.00 mm, vias 2 -> 0
- net COL4_r: track 155.1 -> 0.00 mm, vias 3 -> 0
- net vcc_r: track 148.1 -> 0.00 mm, vias 6 -> 0
- net ROW1: track 141.6 -> 0.00 mm
- net ROW2: track 137.8 -> 0.00 mm, vias 2 -> 0
- net COL0: track 135.6 -> 0.00 mm
- net vcc: track 133.4 -> 0.00 mm, vias 3 -> 0
- net COL3_r: track 132.8 -> 0.00 mm, vias 6 -> 0
- net ROW0: track 130.7 -> 0.00 mm, vias 1 -> 0
- net IPD_DATA_r: track 121.7 -> 0.00 mm, vias 1 -> 0
- net IPD_RST_r: track 118.3 -> 0.00 mm, vias 2 -> 0
- net ROW0_r: track 116.8 -> 0.00 mm
- net IPD_CLK: track 116.7 -> 0.00 mm, vias 3 -> 0
- net ROW2_r: track 114.4 -> 0.00 mm
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- removed copper zone on B.Cu, net gnd
- removed copper zone on F.Cu, net gnd
- removed copper zone on B.Cu, net gnd_r
- removed copper zone on F.Cu, net gnd_r

Commit message: feat: basic shematics
Parts:
- removed Bat+1, Bat+r1, BatGND1, BatGNDr1: MountingHole_Pad, kbd:1pin_conn
- removed the J1 at (253.6, 101.3)
- added BT3: Battery, keystone82:batteryHolder_10440_Keystone_82, F.Cu at (174.3, 118.9)
- added D35: 1N4148W, Diode_SMD:D_SOD-123, F.Cu at (122.9, 150.1)
- added D36: 1N4148W, Diode_SMD:D_SOD-123, F.Cu at (254.8, -43.6)
- added J1: batt_conn, Connector_PinHeader_2.54mm:PinHeader_1x02_P2.54mm_Vertical, F.Cu at (150.8, 111.1)
- added J1: batt_conn, Connector_PinHeader_2.54mm:PinHeader_1x02_P2.54mm_Vertical, F.Cu at (150.9, 126.7)
- added J10: batt_conn, Connector_PinHeader_2.54mm:PinHeader_1x02_P2.54mm_Vertical, F.Cu at (249.5, -43.0)
- added J11: batt_conn, Connector_PinSocket_2.54mm:PinSocket_1x02_P2.54mm_Vertical, F.Cu at (249.5, -50.1)
- added J12: batt_conn, Connector_PinSocket_2.54mm:PinSocket_1x02_P2.54mm_Vertical, F.Cu at (254.1, -50.1)
- added J13: nfc, Connector_PinSocket_2.54mm:PinSocket_1x02_P2.54mm_Vertical, F.Cu at (228.0, -10.3)
- added J14: nfc, Connector_PinSocket_2.54mm:PinSocket_1x02_P2.54mm_Vertical, F.Cu at (242.7, -4.11)
- added J15: extra_btn, Connector_PinSocket_2.54mm:PinSocket_1x02_P2.54mm_Vertical, F.Cu at (151.5, -23.1)
- added J16: extra_btn, Connector_PinSocket_2.54mm:PinSocket_1x02_P2.54mm_Vertical, F.Cu at (156.1, -23.1)
- added J17: TP_thumb_r, trackpoint:trackpoint_mount_t460s_offset, F.Cu at (90.7, 97.2)
- added J18: TP_thumb, trackpoint:trackpoint_mount_t460s_offset, F.Cu at (205.7, 97.2)
- added J19: TP_index_r, trackpoint:trackpoint_mount_t460s_offset, F.Cu at (70.5, 56.6)
- added J2: batt_conn, Connector_PinHeader_2.54mm:PinHeader_1x02_P2.54mm_Vertical, F.Cu at (366.2, -6.36)
- added J20: TP_index, trackpoint:trackpoint_mount_t460s_offset, F.Cu at (225.6, 57.0)
- added J7: batt_conn, Connector_PinSocket_2.54mm:PinSocket_1x02_P2.54mm_Vertical, F.Cu at (244.5, 53.6)
- added J7: batt_conn, Connector_PinSocket_2.54mm:PinSocket_1x02_P2.54mm_Vertical, F.Cu at (244.8, 88.3)
- added J8: batt_conn, Connector_PinHeader_2.54mm:PinHeader_1x02_P2.54mm_Vertical, F.Cu at (192.9, 111.1)
- added J8: batt_conn, Connector_PinHeader_2.54mm:PinHeader_1x02_P2.54mm_Vertical, F.Cu at (192.8, 126.6)
- added J9: batt_conn, Connector_PinSocket_2.54mm:PinSocket_1x02_P2.54mm_Vertical, F.Cu at (260.3, 46.4)
- added J9: batt_conn, Connector_PinSocket_2.54mm:PinSocket_1x02_P2.54mm_Vertical, F.Cu at (260.3, 88.4)
- added U2: SeeeduinoXIAO_BLE, xiao:XIAO-nRF52840-SMD, F.Cu at (174.2, -0.32)
- added U4: 74HC595, sn74hc595dr:D0016A_N, B.Cu at (160.9, 43.3)
- BT1: value 1044 -> Battery; footprint 1044:BAT_1044 -> keystone82:batteryHolder_10440_Keystone_82
- SW1, SW10, SW10_r1, SW11, SW11_r1, SW12, SW12_r1, SW13, SW13_r1, SW14, SW14_r1, SW15, SW15_r1, SW16, SW16_r1, SW17, SW17_r1, SW1_r1, SW2, SW2_r1, SW3, SW3_r1, SW4, SW4_r1, SW5, SW5_r1, SW6, SW6_r1, SW7, SW7_r1, SW8, SW8_r1, SW9, SW9_r1: footprint choc_switch_3d:SW_Hotswap_Kailh_Choc_V1_tweaked -> choc_switch:SW_Hotswap_Kailh_Choc_V1_tweaked_no_clickbar
- U1: value ProMicro-kbd -> SeeeduinoXIAO_BLE; footprint Arduino:Sparkfun_Pro_Micro -> xiao:XIAO-nRF52840-SMD; moved to F.Cu
- U3: value Seeed Studio XIAO SAMD21 -> 74HC595; footprint xiao:XIAO-nRF52840-SMD -> sn74hc595dr:D0016A_N; moved to B.Cu
- moved BT1 265.4 mm to (175.0, -32.0), turned to 0 degrees
- moved U3 133.9 mm to (139.4, 45.1), turned to 180 degrees
- moved U1 95.1 mm to (196.4, 0.06)
- moved SW_POWER1 52.5 mm to (302.7, 29.3)
- moved RSW1 44.3 mm to (289.5, 98.4), turned to 0 degrees
- moved D29 13.1 mm to (57.5, 78.3)
- moved D24 12.7 mm to (57.2, 62.5)
- moved D5 12.5 mm to (238.7, 52.2)
- moved J4 10.4 mm to (258.3, 94.7)
- moved D19 9.90 mm to (57.1, 46.3)
- moved D4 9.87 mm to (213.2, 50.7)
- moved D10 7.47 mm to (237.5, 62.5)
- moved J6 2.49 mm to (118.4, 33.3)
- turned SW10_r1 to 180 degrees
- turned SW15_r1 to 180 degrees
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Connections:
- D11 pad 1: ROW2 -> ROW1
- D12 pad 1: ROW2 -> ROW1
- D16 pad 1: ROW3 -> ROW2
- D17 pad 1: ROW3 -> ROW2
- D23 pad 1: ROW1_r -> ROW0_r
- D28 pad 1: ROW2_r -> ROW1_r
- D29 pad 1: ROW2_r -> ROW1_r
- D33 pad 1: ROW3_r -> ROW2_r
- D34 pad 1: ROW3_r -> ROW2_r
- D6 pad 1: ROW1 -> ROW0
- J3 pad 10: unconnected-(J3-Pin_10-Pad10) -> IPD_RST
- J3 pad 11: unconnected-(J3-Pin_11-Pad11) -> IPD_DATA
- J3 pad 12: unconnected-(J3-Pin_12-Pad12) -> vcc
- J3 pad 5: unconnected-(J3-Pin_5-Pad5) -> IPD_CLK
- J3 pad 6: unconnected-(J3-Pin_6-Pad6) -> gnd
- J6 pad 10: unconnected-(J6-Pin_10-Pad10) -> IPD_RST_r
- J6 pad 11: unconnected-(J6-Pin_11-Pad11) -> IPD_DATA_r
- J6 pad 12: unconnected-(J6-Pin_12-Pad12) -> vcc_r
- J6 pad 5: unconnected-(J6-Pin_5-Pad5) -> IPD_CLK_r
- J6 pad 6: unconnected-(J6-Pin_6-Pad6) -> gnd_r
- SW10 pad 1: COL4 -> COL3
- SW10_r1 pad 1: COL0_r -> COL3_r
- SW10_r1 pad 2: Net-(D23-A) -> Net-(D27-A)
- SW11 pad 1: COL0 -> COL4
- SW11_r1 pad 2: Net-(D32-A) -> Net-(D28-A)
- SW12 pad 1: COL1 -> COL5
- SW12_r1 pad 1: COL3_r -> COL5_r
- SW12_r1 pad 2: Net-(D31-A) -> Net-(D29-A)
- SW13 pad 1: COL2 -> COL0
- SW13_r1 pad 1: COL2_r -> COL0_r
- SW14 pad 1: COL3 -> COL1
- SW14_r1 pad 2: Net-(D29-A) -> Net-(D31-A)
- SW15 pad 1: COL4 -> COL2
- SW15_r1 pad 1: COL0_r -> COL2_r
- SW15_r1 pad 2: Net-(D28-A) -> Net-(D32-A)
- SW16_r1 pad 1: COL1_r -> COL3_r
- SW16_r1 pad 2: Net-(D34-A) -> Net-(D33-A)
- SW17_r1 pad 1: COL0_r -> COL4_r
- SW17_r1 pad 2: Net-(D33-A) -> Net-(D34-A)
- SW1_r1 pad 1: COL4_r -> COL0_r
- SW1_r1 pad 2: Net-(D22-A) -> Net-(D18-A)
- SW2_r1 pad 1: COL3_r -> COL1_r
- SW2_r1 pad 2: Net-(D21-A) -> Net-(D19-A)
- SW4_r1 pad 1: COL1_r -> COL3_r
- SW4_r1 pad 2: Net-(D19-A) -> Net-(D21-A)
- SW5_r1 pad 1: COL0_r -> COL4_r
- SW5_r1 pad 2: Net-(D18-A) -> Net-(D22-A)
- SW6 pad 1: COL0 -> COL5
- SW6_r1 pad 1: COL4_r -> COL5_r
- SW6_r1 pad 2: Net-(D27-A) -> Net-(D23-A)
- SW7 pad 1: COL1 -> COL0
- SW7_r1 pad 1: COL3_r -> COL0_r
- SW7_r1 pad 2: Net-(D26-A) -> Net-(D24-A)
- SW8 pad 1: COL2 -> COL1
- SW8_r1 pad 1: COL2_r -> COL1_r
- SW9 pad 1: COL3 -> COL2
- SW9_r1 pad 1: COL1_r -> COL2_r
- SW9_r1 pad 2: Net-(D24-A) -> Net-(D26-A)
- U1 pad 1: CS -> ROW0
- U1 pad 10: ROW1 -> MOSI
- U1 pad 11: ROW2 -> MISO
- U1 pad 12: ROW3 -> vcc
- U1 pad 13: COL1 -> gnd
- U1 pad 14: COL0 -> unconnected-(U1-5V-Pad14)
- U1 pad 15: COL2 -> reset
- U1 pad 16: COL3 -> raw
- U1 pad 17: COL4 -> Net-(J13-Pin_2)
- U1 pad 18: GPIO1 -> Net-(J13-Pin_1)
- U1 pad 19: IPD_RST -> (no net)
- U1 pad 2: MISO -> CS
- U1 pad 20: GPIO2 -> (no net)
- U1 pad 21: vcc -> (no net)
- U1 pad 22: reset -> (no net)
- U1 pad 3: gnd -> ROW1
- U1 pad 4: gnd -> ROW2
- U1 pad 5: MOSI -> IPD_DATA
- U1 pad 6: SCK -> IPD_CLK
- U1 pad 7: IPD_DATA -> IPD_RST
- U1 pad 8: IPD_CLK -> SR_CS
- U1 pad 9: ROW0 -> SCK
- U3 pad 1: unconnected-(U3-PA02_A0_D0-Pad1) -> COL0_r
- U3 pad 10: unconnected-(U3-PA5_A9_D9_MISO-Pad10) -> Net-(U3-VCC)
- U3 pad 11: unconnected-(U3-PA6_A10_D10_MOSI-Pad11) -> SCK_r
- U3 pad 12: unconnected-(U3-3V3-Pad12) -> SR_CS_r
- U3 pad 13: unconnected-(U3-GND-Pad13) -> gnd_r
- U3 pad 14: unconnected-(U3-5V-Pad14) -> MOSI_r
- U3 pad 15: unconnected-(U3-5V-Pad15) -> COL2_r
- U3 pad 16: unconnected-(U3-GND-Pad16) -> Net-(U3-VCC)
- U3 pad 2: unconnected-(U3-PA4_A1_D1-Pad2) -> COL1_r
- U3 pad 3: unconnected-(U3-PA10_A2_D2-Pad3) -> COL3_r
- U3 pad 4: unconnected-(U3-PA11_A3_D3-Pad4) -> COL5_r
- U3 pad 5: unconnected-(U3-PA8_A4_D4_SDA-Pad5) -> COL4_r
- U3 pad 8: unconnected-(U3-PB09_A7_D7_RX-Pad8) -> gnd_r
Other:
- board size 246.8 x 97.3 mm -> 240.6 x 100.7 mm
- board text removed: "BT+"
- board text removed: "Do not solder board to this side"

Commit message: feat: more pcb item placements
Parts:
- removed BT3: Battery, keystone82:batteryHolder_10440_Keystone_82
- removed the J11 at (249.5, -50.1)
- removed the J2 at (366.2, -6.36)
- removed the J7 at (244.5, 53.6)
- removed the J7 at (244.8, 88.3)
- removed the J9 at (260.3, 46.4)
- removed the J9 at (260.3, 88.4)
- added BT2: Battery_Cell, keystone82:batteryHolder_10440_Keystone_82, F.Cu at (174.3, 119.6)
- added G***: LOGO, silkscreens:plus_circle, F.Cu at (52.0, 60.5)
- added G***: LOGO, silkscreens:plus_circle, F.Cu at (244.4, 61.1)
- added G***: LOGO, silkscreens:plus_circle, F.Cu at (131.7, 119.8)
- added G***: LOGO, silkscreens:plus_circle, F.Cu at (164.5, 119.7)
- added J10: batt_pin, Connector_PinHeader_2.54mm:PinHeader_1x02_P2.54mm_Vertical, F.Cu at (138.2, 111.9)
- added J11: batt_socket, Connector_PinSocket_2.54mm:PinSocket_1x02_P2.54mm_Vertical, F.Cu at (51.0, 88.4)
- added J11: batt_socket, Connector_PinSocket_2.54mm:PinSocket_1x02_P2.54mm_Vertical, F.Cu at (35.6, 88.4)
- added J12: batt_socket, Connector_PinSocket_2.54mm:PinSocket_1x02_P2.54mm_Vertical, F.Cu at (51.2, 54.9)
- added J2: batt_pin, Connector_PinHeader_2.54mm:PinHeader_1x02_P2.54mm_Vertical, F.Cu at (104.6, 111.9)
- added J2: batt_pin, Connector_PinHeader_2.54mm:PinHeader_1x02_P2.54mm_Vertical, F.Cu at (104.6, 127.4)
- added J7: batt_socket, Connector_PinSocket_2.54mm:PinSocket_1x02_P2.54mm_Vertical, F.Cu at (260.9, 88.5)
- added J7: batt_socket, Connector_PinSocket_2.54mm:PinSocket_1x02_P2.54mm_Vertical, F.Cu at (245.3, 88.5)
- added J9: batt_socket, Connector_PinSocket_2.54mm:PinSocket_1x02_P2.54mm_Vertical, F.Cu at (245.1, 54.9)
- added J9: batt_socket, Connector_PinSocket_2.54mm:PinSocket_1x02_P2.54mm_Vertical, F.Cu at (260.7, 54.9)
- added SW11: SW_Push, choc_switch:SW_Hotswap_Kailh_Choc_V1_tweaked_no_clickbar, F.Cu at (162.7, 94.3)
- added SW11_r1: SW_Push, choc_switch:SW_Hotswap_Kailh_Choc_V1_tweaked_no_clickbar, F.Cu at (133.8, 94.3)
- added mouse-bite-2mm-slot1: VAL**, Duckyb-Parts:mouse-bite-5mm-slot-with-space-for-track, F.Cu at (147.8, 113.3)
- added mouse-bite-2mm-slot1: VAL**, Duckyb-Parts:mouse-bite-5mm-slot-with-space-for-track, F.Cu at (154.1, 108.8)
- added mouse-bite-2mm-slot1: VAL**, Duckyb-Parts:mouse-bite-5mm-slot-with-space-for-track, F.Cu at (170.6, 108.9)
- added mouse-bite-2mm-slot1: VAL**, Duckyb-Parts:mouse-bite-5mm-slot-with-space-for-track, F.Cu at (147.8, 125.8)
- BT1: value Battery -> Battery_Cell
- J1 (x2), J10, J8 (x2): value batt_conn -> batt_pin
- J12: value batt_conn -> batt_socket
- RSW1, RSW2: footprint reset_switch:PTS636SP43LFS -> Button_Switch_SMD:Panasonic_EVQPUL_EVQPUC; moved to B.Cu
- SW6, SW6_r1: footprint choc_switch:SW_Hotswap_Kailh_Choc_V1_tweaked_no_clickbar -> choc_switch_3d:SW_Hotswap_Kailh_Choc_V1_tweaked_23du
- moved J12 242.4 mm to (35.6, 54.9), turned to 180 degrees
- moved J10 203.6 mm to (138.2, 127.5), turned to 90 degrees
- moved BT1 160.9 mm to (121.5, 119.7), turned to 180 degrees
- moved RSW1 150.3 mm to (155.8, 29.7), turned to 180 degrees
- moved RSW2 138.6 mm to (141.4, 30.1), turned to 180 degrees
- moved D36 138.0 mm to (203.8, 84.7), turned to 180 degrees
- moved SW_POWER1 136.5 mm to (166.2, 29.4)
- moved J16 128.3 mm to (91.5, 87.7), turned to 90 degrees
- moved J14 122.7 mm to (132.9, 50.7), turned to 90 degrees
- moved J15 122.4 mm to (203.6, 87.6), turned to 90 degrees
- moved J13 91.0 mm to (160.3, 50.6), turned to 90 degrees
- moved SW_POWERR1 90.8 mm to (130.2, 29.3)
- moved D35 72.5 mm to (91.9, 84.5), turned to 180 degrees
- moved U2 55.3 mm to (134.8, 38.5)
- moved U1 51.7 mm to (161.8, 38.4)
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Connections:
- J10 pad 1: BT+ -> BT+_r
- J10 pad 2: BT+ -> BT+_r
- J12 pad 1: BT+ -> BT+_r
- J12 pad 2: BT+ -> BT+_r
Other:
- board size 240.6 x 100.7 mm -> 234.4 x 101.4 mm
- board text added: "-"
- board text added: "Locealda V1.0.0"
- board text removed: "B+"
- board text removed: "B-"
- board text removed: "Face down"
- board text removed: "Seahorse V2.0.0"

Commit message: feat: xiao bottom access
Parts:
- removed J13, J14: nfc, Connector_PinSocket_2.54mm:PinSocket_1x02_P2.54mm_Vertical
- added REF**: TestPoint_Pad_D1.0mm, TestPoint:TestPoint_Pad_D1.0mm, B.Cu at (131.4, 22.5)
- D35, D36: moved to B.Cu
- mouse-bite-2mm-slot1: value VAL** -> (none)
- mouse-bite-2mm-slot1: value VAL** -> 1
- moved SW_POWER1 66.5 mm to (183.2, 93.7), turned to 0 degrees
- moved SW_POWERR1 66.4 mm to (113.2, 93.5), turned to 0 degrees
- moved RSW2 43.6 mm to (97.8, 31.1)
- moved RSW1 42.9 mm to (198.7, 31.1)
- moved D23 9.84 mm to (84.0, 66.5)
- moved U4 5.98 mm to (160.5, 46.7)
- moved U3 5.60 mm to (133.3, 46.2), turned to 0 degrees
- moved D9 2.67 mm to (210.9, 60.2)
- moved U1 0.09 mm to (161.7, 38.5)
- turned D35 to 0 degrees
- turned D36 to 0 degrees
Connections:
- J5 pad 5: CS_R -> CS_r
- J7 pad 1: (no net) -> gnd
- J7 pad 2: (no net) -> gnd
- J9 pad 1: (no net) -> BT+
- J9 pad 2: (no net) -> BT+
- U2 pad 16: raw_batt+_r -> BT+_r
Routing:
- net BT+_r: track 0.00 -> 128.8 mm, vias 0 -> 2
- net vcc_r: track 0.00 -> 12.4 mm, vias 0 -> 1
- net IPD_DATA_r: track 0.00 -> 11.4 mm, vias 0 -> 1
- net gnd_r: track 0.00 -> 5.08 mm, vias 0 -> 1
- net ROW1_r: track 0.00 -> 2.14 mm, vias 0 -> 1
- net CS_r: track 0.00 -> 2.12 mm, vias 0 -> 1
- net unconnected-(U2-5V-Pad14): vias 0 -> 1
- net reset_r: vias 0 -> 1
- net reset: vias 0 -> 1
- net raw: vias 0 -> 1
- net nfc_2_r: vias 0 -> 1
- net nfc_1_r: vias 0 -> 1
- net SR_CS_r: vias 0 -> 1
- net SCK_r: vias 0 -> 1
- net ROW2_r: vias 0 -> 1
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Other:
- outline, holes or cut-outs redrawn

Commit message: feat: remove battery
Parts:
- removed BT1, BT2: Battery_Cell, keystone82:batteryHolder_10440_Keystone_82
- removed G*** (x4): LOGO, silkscreens:plus_circle
- removed the J1 at (188.9, 127.4)
- removed the J1 at (188.9, 111.8)
- removed J10 (x2), J2 (x2), J8 (x2): batt_pin, Connector_PinHeader_2.54mm:PinHeader_1x02_P2.54mm_Vertical
- removed J11 (x2), J12 (x2), J7 (x2), J9 (x2): batt_socket, Connector_PinSocket_2.54mm:PinSocket_1x02_P2.54mm_Vertical
- removed REF**: TestPoint_Pad_D1.0mm, TestPoint:TestPoint_Pad_D1.0mm
- removed the mouse-bite-2mm-slot1 at (147.8, 113.3)
- removed the mouse-bite-2mm-slot1 at (154.1, 108.8)
- removed the mouse-bite-2mm-slot1 at (170.6, 108.9)
- removed the mouse-bite-2mm-slot1 at (147.8, 125.8)
- added J1: batt_jst_conn, Connector_JST:JST_PH_S2B-PH-K_1x02_P2.00mm_Horizontal, B.Cu at (59.1, 96.5)
- added J13: nfc, Connector_PinSocket_2.54mm:PinSocket_1x02_P2.54mm_Vertical, F.Cu at (135.4, 9.90)
- added J14: nfc, Connector_PinSocket_2.54mm:PinSocket_1x02_P2.54mm_Vertical, F.Cu at (172.6, 8.05)
- added J21: batt_jst_conn_r, Connector_JST:JST_PH_S2B-PH-K_1x02_P2.00mm_Horizontal, F.Cu at (251.3, 89.4)
- moved U2 89.6 mm to (46.3, 51.8)
- moved SW_POWER1 73.7 mm to (256.8, 89.6), turned to 90 degrees
- moved RSW2 65.2 mm to (116.6, 93.4), turned to 0 degrees
- moved SW_POWERR1 61.3 mm to (118.1, 32.5), turned to 180 degrees
- moved U4 54.5 mm to (178.8, 98.0), turned to -90 degrees
- moved J6 17.8 mm to (136.2, 34.9)
- moved D24 8.47 mm to (65.7, 62.0)
- moved D29 7.95 mm to (65.9, 87.3)
- moved D3 5.92 mm to (199.7, 36.4)
- moved U3 4.32 mm to (137.1, 48.4), turned to 90 degrees
- moved J5 3.14 mm to (41.8, 96.3)
- moved D18 3.00 mm to (84.0, 50.5)
- moved D19 3.00 mm to (60.1, 46.3)
- moved D20 3.00 mm to (96.3, 45.9)
- moved D21 3.00 mm to (114.3, 42.9)
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Connections:
- U3 pad 10: Net-(U3-VCC) -> vcc_r
- U3 pad 16: Net-(U3-VCC) -> vcc_r
Routing:
- net BT+_r: track 128.8 -> 0.00 mm, vias 2 -> 1
- net vcc_r: track 12.4 -> 0.00 mm, vias 1 -> 0
- net IPD_DATA_r: track 11.4 -> 0.00 mm, vias 1 -> 0
- net gnd_r: track 5.08 -> 0.00 mm, vias 1 -> 0
- net ROW1_r: track 2.14 -> 0.00 mm, vias 1 -> 0
- net CS_r: track 2.12 -> 0.00 mm, vias 1 -> 0
- net unconnected-(U2-5V-Pad14): vias 1 -> 0
- net reset: vias 1 -> 0
- net raw: vias 1 -> 0
- net nfc_2_r: vias 1 -> 0
- net nfc_1_r: vias 1 -> 0
- net SR_CS_r: vias 1 -> 0
- net SCK_r: vias 1 -> 0
- net ROW2_r: vias 1 -> 0
- net ROW0_r: vias 1 -> 0
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Other:
- board size 234.4 x 101.4 mm -> 221.7 x 93.3 mm
- board text removed: "-"
- board text removed: "Locealda V1.0.0"

Commit message: feat: cleanup footprint shape
Parts:
- removed mouse-bite-2mm-slot1: VAL**, Duckyb-Parts:mouse-bite-5mm-slot-with-space-for-track
- removed mouse-bite-2mm-slot1: 1, Duckyb-Parts:mouse-bite-5mm-slot-with-space-for-track
- J21: moved to B.Cu
- moved J14 131.4 mm to (55.1, 66.7), turned to 180 degrees
- moved J13 120.3 mm to (241.4, 66.8), turned to 180 degrees
- moved SW_POWER1 97.0 mm to (178.4, 32.5), turned to 180 degrees
- moved U1 92.2 mm to (250.3, 51.8)
- moved RSW1 64.3 mm to (179.9, 93.5), turned to 0 degrees
- moved U4 53.2 mm to (159.4, 48.4)
- moved J3 19.8 mm to (160.3, 34.9)
- moved J21 16.4 mm to (236.5, 96.6), turned to -30 degrees
- moved J15 1.06 mm to (202.0, 87.6), turned to -90 degrees
- moved J4 0.42 mm to (254.7, 96.3)
- moved J18 0.08 mm to (203.0, 97.3)
Routing:
- net reset_r: vias 1 -> 2
- net BT+_r: vias 1 -> 2
Other:
- board size 221.7 x 93.3 mm -> 223.3 x 90.6 mm
- board text removed: "By N8"
- board text removed: "LEFT"

Commit message: wip: begin routing
Parts:
- removed J13, J14: nfc, Connector_PinSocket_2.54mm:PinSocket_1x02_P2.54mm_Vertical
- added mouse-bite-2mm-slot1: VAL**, Duckyb-Parts:mouse-bite-5mm-slot-with-space-for-track, F.Cu at (148.2, 52.2)
- added mouse-bite-2mm-slot1: VAL**, Duckyb-Parts:mouse-bite-5mm-slot-with-space-for-track, F.Cu at (148.3, 79.5)
- moved U3 92.7 mm to (44.8, 56.7)
- moved U4 89.8 mm to (248.8, 56.7)
- moved D3 15.1 mm to (185.6, 41.8)
- moved J3 6.92 mm to (159.8, 41.8)
- moved D5 6.77 mm to (229.3, 53.1)
- moved J6 6.70 mm to (136.7, 41.6)
- moved SW_POWER1 4.27 mm to (182.1, 34.6)
- moved SW_POWERR1 3.63 mm to (115.1, 34.5)
Connections:
- U1 pad 17: Net-(J13-Pin_2) -> unconnected-(U1-J13-pin_2-Pad17)
- U1 pad 18: Net-(J13-Pin_1) -> unconnected-(U1-J13-pin_1-Pad18)
- U4 pad 10: Net-(U4-VCC) -> vcc
- U4 pad 16: Net-(U4-VCC) -> vcc
Routing:
- net vcc: track 0.00 -> 196.3 mm, vias 0 -> 8
- net IPD_RST: track 0.00 -> 133.4 mm, vias 0 -> 4
- net IPD_DATA: track 0.00 -> 131.0 mm, vias 0 -> 2
- net IPD_CLK: track 0.00 -> 128.1 mm, vias 0 -> 6
- net gnd: track 0.00 -> 126.0 mm, vias 0 -> 9
- net raw: track 0.00 -> 71.2 mm, vias 0 -> 1
- net CS: track 0.00 -> 70.9 mm
- net SCK: track 0.00 -> 57.6 mm, vias 0 -> 2
- net MOSI: track 0.00 -> 56.6 mm, vias 0 -> 2
- net COL3: track 0.00 -> 49.8 mm, vias 0 -> 1
- net COL0: track 0.00 -> 48.8 mm, vias 0 -> 1
- net vcc_r: track 0.00 -> 37.2 mm, vias 0 -> 5
- net COL4: track 0.00 -> 30.6 mm, vias 0 -> 2
- net COL2: track 0.00 -> 9.99 mm
- net SR_CS: track 0.00 -> 9.85 mm, vias 0 -> 2
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Other:
- board size 223.3 x 90.6 mm -> 223.3 x 88.9 mm
