File: loce_alda_v1/loce_alda_v1_0_0.kicad_sch (KiCad schematic)
At the start: 90 parts, among them J1 batt_jst_conn, J15 extra_btn, J16 extra_btn, J17 TP_thumb_r, J18 TP_thumb, J19 TP_index_r, J20 TP_index, J21 batt_jst_conn_r, J3 track_point_left, J4 niceview_left, J5 niceview_right, J6 track_point_right, SW1 SW_Push, SW10 SW_Push, SW10_r1 SW_Push, SW11 SW_Push, SW11_r1 SW_Push, SW12 SW_Push, SW12_r1 SW_Push, SW13 SW_Push, SW13_r1 SW_Push, SW14 SW_Push, SW14_r1 SW_Push, SW15 SW_Push, SW15_r1 SW_Push, SW16 SW_Push, SW16_r1 SW_Push, SW17 SW_Push, SW17_r1 SW_Push, SW1_r1 SW_Push, SW2 SW_Push, SW2_r1 SW_Push, SW3 SW_Push, SW3_r1 SW_Push, SW4 SW_Push, SW4_r1 SW_Push, SW5 SW_Push, SW5_r1 SW_Push, SW6 SW_Push, SW6_r1 SW_Push, SW7 SW_Push, SW7_r1 SW_Push, SW8 SW_Push, SW8_r1 SW_Push, SW9 SW_Push, SW9_r1 SW_Push, U1 SeeeduinoXIAO_BLE, U2 SeeeduinoXIAO_BLE, U3 74HC595, U4 74HC595

Commit message: feat: wire the loce alda
Connections:
- net BT+: now also J21.2 (Pin_2); no longer J21.1 (Pin_1)
- net BT+_r: now also J1.2 (Pin_2); no longer J1.1 (Pin_1), U2.16 (BAT+)
- net gnd: now also J21.1 (Pin_1); no longer J21.2 (Pin_2)
- net gnd_r: now also J1.1 (Pin_1); no longer J1.2 (Pin_2)
- net raw_r: now also U2.16 (BAT+)
- net nfc_1_r: no longer names the net of U2.18 (J13-pin_1)
- net nfc_2_r: no longer names the net of U2.17 (J13-pin_2)
- no-connect marks 12 -> 20
Changed lines of the file:
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@@
 	)
 	(no_connect
+		(at 270.51 36.83)
+	)
+	(no_connect
 		(at 46.99 313.69)
 	)
@@
 	)
 	(no_connect
+		(at 294.64 48.26)
+	)
+	(no_connect
+		(at 62.23 36.83)
+	)
+	(no_connect
+		(at 273.05 36.83)
+	)
+	(no_connect
+		(at 387.35 120.65)
+	)
+	(no_connect
 		(at 93.98 203.2)
 	)
@@
 	)
 	(no_connect
+		(at 387.35 115.57)
+	)
+	(no_connect
 		(at 86.36 49.53)
 	)
 	(no_connect
+		(at 64.77 36.83)
+	)
+	(no_connect
+		(at 387.35 113.03)
+	)
+	(no_connect
 		(at 45.72 303.53)
 	)
@@
 		(at 33.02 304.8)
 	)
+	(bus_entry
+		(at 431.8 92.71)
+		(size 2.54 2.54)
+		(stroke
+			(width 0)
+			(type default)
+		)
+	)
+	(bus_entry
+		(at 74.93 165.1)
+		(size 2.54 2.54)
+		(stroke
+			(width 0)
+			(type default)
+		)
+	)
 	(wire
 		(pts
@@
 	(wire
 		(pts
-			(xy 83.82 167.64) (xy 68.58 167.64)
+			(xy 83.82 167.64) (xy 77.47 167.64)
 		)
 		(stroke
@@
 	(wire
 		(pts
+			(xy 77.47 167.64) (xy 68.58 167.64)
+		)
+		(stroke
+			(width 0)
+			(type default)
+		)
+	)
+	(wire
+		(pts
 			(xy 83.82 165.1) (xy 83.82 167.64)
 		)
@@
 		)
 	)
-	(global_label "nfc_2_r"
-		(shape input)
-		(at 273.05 36.83 90)
-		(fields_autoplaced yes)
-		(effects
-			(font
-				(size 1.27 1.27)
-			)
-			(justify left)
-		)
-		(property "Intersheetrefs" "${INTERSHEET_REFS}"
-			(at 273.05 26.9506 90)
-			(effects
-				(font
-					(size 1.27 1.27)
-				)
-				(justify left)
-				(hide yes)
-			)
-		)
-	)
 	(global_label "SCK"
 		(shape input)
@@
 		)
 	)
+	(global_label "BT+_r"
+		(shape input)
+		(at 365.76 63.5 0)
+		(fields_autoplaced yes)
+		(effects
+			(font
+				(size 1.27 1.27)
+			)
+			(justify left)
+		)
+		(property "Intersheetrefs" "${INTERSHEET_REFS}"
+			(at 374.309 63.5 0)
+			(effects
+				(font
+					(size 1.27 1.27)
+				)
+				(justify left)
+				(hide yes)
+			)
+		)
+	)
 	(global_label "COL0"
 		(shape input)
@@
 		)
 	)
-	(global_label "BT+"
+	(global_label "MOSI_r"
 		(shape input)
-		(at 165.1 35.56 0)
+		(at 297.18 59.69 0)
 		(fields_autoplaced yes)
 		(effects
@@
 		)
 		(property "Intersheetrefs" "${INTERSHEET_REFS}"
-			(at 171.8952 35.56 0)
+			(at 306.5152 59.69 0)
 			(effects
 				(font
@@
 		)
 	)
-	(global_label "MOSI_r"
+	(global_label "BT+"
 		(shape input)
-		(at 297.18 59.69 0)
+		(at 165.1 38.1 0)
 		(fields_autoplaced yes)
 		(effects
@@
 		)
 		(property "Intersheetrefs" "${INTERSHEET_REFS}"
-			(at 306.5152 59.69 0)
+			(at 171.8952 38.1 0)
 			(effects
 				(font
@@
 		)
 	)
-	(global_label "nfc_1_r"
-		(shape input)
-		(at 270.51 36.83 90)
-		(fields_autoplaced yes)
-		(effects
-			(font
-				(size 1.27 1.27)
-			)
-			(justify left)
-		)
-		(property "Intersheetrefs" "${INTERSHEET_REFS}"
-			(at 270.51 26.9506 90)
-			(effects
-				(font
-					(size 1.27 1.27)
-				)
-				(justify left)
-				(hide yes)
-			)
-		)
-	)
 	(global_label "COL1"
 		(shape input)
@@
 		)
 	)
-	(global_label "gnd"
-		(shape input)
-		(at 165.1 38.1 0)
-		(fields_autoplaced yes)
-		(effects
-			(font
-				(size 1.27 1.27)
-			)
-			(justify left)
-		)
-		(property "Intersheetrefs" "${INTERSHEET_REFS}"
-			(at 171.5322 38.1 0)
-			(effects
-				(font
-					(size 1.27 1.27)
-				)
-				(justify left)
-				(hide yes)
-			)
-		)
-	)
 	(global_label "IPD_CLK_r"
 		(shape input)
@@
 		)
 	)
-	(global_label "BT+_r"
-		(shape input)
-		(at 365.76 60.96 0)
-		(fields_autoplaced yes)
-		(effects
-			(font
-				(size 1.27 1.27)
-			)
-			(justify left)
-		)
-		(property "Intersheetrefs" "${INTERSHEET_REFS}"
-			(at 374.309 60.96 0)
-			(effects
-				(font
-					(size 1.27 1.27)
-				)
-				(justify left)
-				(hide yes)
-			)
-		)
-	)
 	(global_label "MOSI"
 		(shape input)
@@
 		)
 	)
-	(global_label "BT+_r"
-		(shape input)
-		(at 280.67 35.56 90)
-		(fields_autoplaced yes)
-		(effects
-			(font
-				(size 1.27 1.27)
-			)
-			(justify left)
-		)
-		(property "Intersheetrefs" "${INTERSHEET_REFS}"
-			(at 280.67 27.011 90)
-			(effects
-				(font
-					(size 1.27 1.27)
-				)
-				(justify left)
-				(hide yes)
-			)
-		)
-	)
 	(global_label "MOSI"
 		(shape input)
@@
 		)
 	)
-	(global_label "gnd_r"
-		(shape input)
-		(at 365.76 63.5 0)
-		(fields_autoplaced yes)
-		(effects
-			(font
-				(size 1.27 1.27)
-			)
-			(justify left)
-		)
-		(property "Intersheetrefs" "${INTERSHEET_REFS}"
-			(at 373.946 63.5 0)
-			(effects
-				(font
-					(size 1.27 1.27)
-				)
-				(justify left)
-				(hide yes)
-			)
-		)
-	)
 	(global_label "ROW0"
 		(shape input)
@@
 		)
 	)
+	(global_label "gnd"
+		(shape input)
+		(at 165.1 35.56 0)
+		(fields_autoplaced yes)
+		(effects
+			(font
+				(size 1.27 1.27)
+			)
+			(justify left)
+		)
+		(property "Intersheetrefs" "${INTERSHEET_REFS}"
+			(at 171.5322 35.56 0)
+			(effects
+				(font
+					(size 1.27 1.27)
+				)
+				(justify left)
+				(hide yes)
+			)
+		)
+	)
 	(global_label "SCK_r"
 		(shape input)
@@
 		)
 	)
+	(global_label "raw_r"
+		(shape input)
+		(at 280.67 35.56 90)
+		(fields_autoplaced yes)
+		(effects
+			(font
+				(size 1.27 1.27)
+			)
+			(justify left)
+		)
+		(property "Intersheetrefs" "${INTERSHEET_REFS}"
+			(at 280.67 27.5553 90)
+			(effects
+				(font
+					(size 1.27 1.27)
+				)
+				(justify left)
+				(hide yes)
+			)
+		)
+	)
 	(global_label "COL3_r"
 		(shape input)
@@
 			(effects
 				(font
+					(size 1.27 1.27)
+				)
+				(justify left)
+				(hide yes)
+			)
+		)
+	)
+	(global_label "gnd_r"
+		(shape input)
+		(at 365.76 60.96 0)
+		(fields_autoplaced yes)
+		(effects
+			(font
+				(size 1.27 1.27)
+			)
+			(justify left)
+		)
+		(property "Intersheetrefs" "${INTERSHEET_REFS}"
+			(at 373.946 60.96 0)
+			(effects
+				(font
